File: Doorbell with External ESP8266.kicad_pcb (KiCad board)
At the start: 4 copper layers, 70 x 50 mm, 28 parts, among them J101 Transformer, J102 From Rectifier, J103 To Rectifier, J104 Chime, J105 Button, K101 Relay, Q101 Q_NMOS_GSD, U101 WeMos_D1_mini, U103 EL817

Commit message: schematic fix
Parts:
- removed REF**: OSHW-Logo2_7.3x6mm_SilkScreen, Symbol:OSHW-Logo2_7.3x6mm_SilkScreen
- removed REF**: KiCad-Logo2_5mm_SilkScreen, Symbol:KiCad-Logo2_5mm_SilkScreen
- moved R105 4.99 mm to (53.1, 47.6), turned to -90 degrees
- moved Q101 0.59 mm to (49.9, 45.8)
Connections:
- Q101 pad 1: GND -> /CHIME
- Q101 pad 2: /CHIME -> GND
Routing:
- net /AC_A: track 44.2 -> 48.3 mm
- net VCC: track 53.9 -> 57.8 mm
- net /CHIME: track 10.1 -> 12.4 mm
- net GND: track 10.1 -> 7.99 mm, vias 6 -> 5
- net /AC_B: track 59.4 -> 61.2 mm
- net /RELAY_LED: track 29.5 -> 28.9 mm
